File: pcb/CD_Cap_brd.sch (EAGLE design)
At the start: 18 parts, among them Q1 IRF3704S, Q2 IRF3704S

Commit message: almost ready for FAB
Parts:
- removed C4: (no value), passives-7351:CAPACITOR0603-N
Connections:
- net B-: no longer C4.1
- net TRIG: no longer C4.2
Changed lines of the file:
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@@
 <part name="R5" library="passives-7351" deviceset="RESISTOR" device="0603-N" value="10k"/>
 <part name="R6" library="passives-7351" deviceset="RESISTOR" device="0603-N" value="10k"/>
-<part name="C4" library="passives-7351" deviceset="CAPACITOR" device="0603-N"/>
 <part name="C6" library="resistor" deviceset="CPOL-EU" device="E10-35"/>
 <part name="C7" library="resistor" deviceset="CPOL-EU" device="E10-35"/>
@@
 <attribute name="VALUE" x="26.67" y="30.48" size="1.778" layer="95" rot="R180"/>
 </instance>
-<instance part="C4" gate="G$1" x="266.7" y="30.48" rot="R180"/>
 <instance part="C6" gate="G$1" x="60.96" y="15.24"/>
 <instance part="C7" gate="G$1" x="67.31" y="15.24"/>
@@
 </segment>
 <segment>
-<pinref part="C4" gate="G$1" pin="1"/>
-<wire x1="266.7" y1="27.94" x2="266.7" y2="25.4" width="0.1524" layer="91"/>
-<label x="266.7" y="25.4" size="1.27" layer="95" rot="R180" xref="yes"/>
-</segment>
-<segment>
 <pinref part="J4" gate="J$1" pin="3"/>
 <wire x1="63.5" y1="114.3" x2="66.04" y2="114.3" width="0.1524" layer="91"/>
@@
 </segment>
 <segment>
-<pinref part="C4" gate="G$1" pin="2"/>
-<wire x1="266.7" y1="35.56" x2="266.7" y2="38.1" width="0.1524" layer="91"/>
-<label x="266.7" y="38.1" size="1.27" layer="95" rot="R180" xref="yes"/>
-</segment>
-<segment>

Commit message: first circuit Fab: Success
Parts:
- U$1, U$2, U$3, U$4: value BIG_PINHEADX1 -> BIG_PINHEADX110-32; device Ians parts:BIG_PINHEADX1 -> _my-parts:BIG_PINHEADX110-32
Changed lines of the file:
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@@
 <part name="J1" library="SparkFun-Connectors" deviceset="M03" device="PTH"/>
 <part name="J2" library="SparkFun-Connectors" deviceset="M03" device="PTH"/>
-<part name="U$1" library="Ians parts" deviceset="BIG_PINHEADX1" device=""/>
-<part name="U$2" library="Ians parts" deviceset="BIG_PINHEADX1" device=""/>
-<part name="U$3" library="Ians parts" deviceset="BIG_PINHEADX1" device=""/>
-<part name="U$4" library="Ians parts" deviceset="BIG_PINHEADX1" device=""/>
+<part name="U$1" library="_my-parts" deviceset="BIG_PINHEADX1" device="10-32"/>
+<part name="U$2" library="_my-parts" deviceset="BIG_PINHEADX1" device="10-32"/>
+<part name="U$3" library="_my-parts" deviceset="BIG_PINHEADX1" device="10-32"/>
+<part name="U$4" library="_my-parts" deviceset="BIG_PINHEADX1" device="10-32"/>
 <part name="J3" library="SparkFun-Connectors" deviceset="M03" device="LOCK"/>
 <part name="J4" library="SparkFun-Connectors" deviceset="M03" device="LOCK"/>
